File: 312628-REV-5.7A/sheets/PRINTER_SERIAL.kicad_sch (KiCad schematic)
At the start: 86 parts, among them CN401 DB25, CN402 DB25, Q401 2N3904, U401 6242, U402 8250, U403 PPC1, U404 MC1488, U405 MC1489

Commit message: update schematics to kicad 7.0.8
Parts:
- renumbered C202 to C401, C202 to C404, C202 to C405, C202 to C406, C202 to C408, C202 to C409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
