File: 312628-REV-5.7A/sheets/VIDEO.kicad_sch (KiCad schematic)
At the start: 88 parts, among them CN203 Jumper_2_Open, CN601 DB 9, CN602 DB 9, CN603 "RCA" Jack, J1 ALEBODGE_RIGHT, Q601 2N3904, Q602 2N3906, U1 74LS04, U601 PVC4, U602 CSG 5720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

Commit message: update schematics to kicad 7.0.8
Parts:
- renumbered C202 to C601, C202 to C602, C202 to C603, C202 to C604, C202 to C605, C202 to C606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
Connections:
- net SW1: now also U1.13; no longer U1.9
- net at U607.23 (A11): now also U1.12; no longer U1.8
- no-connect marks 10 -> 8
