File: 312628-REV-6C/sheets/EXPANSION.kicad_sch (KiCad schematic)
At the start: 43 parts, among them CN501 Bus_ISA_8bit, CN502 Bus_ISA_8bit, CN503 Bus_ISA_8bit, U111 74LS125

Commit message: Update Schematics to KiCad V8
Parts:
- renumbered R206 to R690, R206 to R691
