File: 312628-REV-6C/sheets/FDD_HDD_BIOS.kicad_sch (KiCad schematic)
At the start: 40 parts, among them CN201 FLOPPY_DISK_CONNECTOR, CN202 IDE, CN203 Jumper_2_Open, U1 74LS04, U2 74LS08, U201 ROM, U202 74LS244, U203 9268, U204 74LS245, U205 74LS245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

Commit message: added PAD204 footprint, update PCB
Parts:
- PAD204: footprint CBM-PC10:PAD101 -> CBM-PC10:PAD204
Changed lines of the file:
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@@
 			)
 		)
-		(property "Footprint" "CBM-PC10:PAD101"
+		(property "Footprint" "CBM-PC10:PAD204"
 			(at 304.8 370.205 0)
 			(effects
