File: 312628-REV-6C/sheets/POWER.kicad_sch (KiCad schematic)
At the start: 95 parts, among them CN504 Jumper_2_Open, CN505 SILPOWER, CN506 POWER, SW501 SW_Push, U1 74LS04, U110 74LS74, U111 74LS125, U2 74LS08, U206 7406, U3 74LS14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

Commit message: Update Schematics to KiCad V8
Parts:
- renumbered U5 to U207, U325 to U313, U326 to U314, U327 to U315, U328 to U316

Commit message: Update to latest KiCad 8.0.7
Update to latest KiCad 8.0.7
Fix wrong value of R504 should be 1K
Parts:
- R504: value 10K -> 1K
Changed lines of the file:
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@@
 		(fields_autoplaced yes)
 		(property "Reference" "R504"
-			(at 212.09 34.925 0)
+			(at 212.09 34.2899 0)
 			(effects
 				(font
@@
 			)
 		)
-		(property "Value" "10K"
-			(at 212.09 37.465 0)
+		(property "Value" "1K"
+			(at 212.09 36.8299 0)
 			(effects
 				(font
