File: 312628-REV-6C/sheets/RAM.kicad_sch (KiCad schematic)
At the start: 21 parts, among them U301 74LS158, U302 74LS158, U303 74LS158, U304 74LS245, U305 44256, U306 44256, U307 44256, U308 44256, U309 4464, U310 4464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

Commit message: Update Schematics to KiCad V8
Parts:
- renumbered R206 to R301
