File: 312628-REV-6C/sheets/CPU.kicad_sch (KiCad schematic)
At the start: 58 parts, among them CN101 SPEAKER, CN102 KEYBRD, Q101 2N3904, U1 74LS04, U101 FE2010, U102 8088, U103 8087, U104 74LS245, U105 74LS373, U106 74LS373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

Commit message: Update Schematics to KiCad V8
Parts:
- renumbered EMI406 to EMI101, EMI406 to EMI102, EMI406 to EMI103, EMI406 to EMI104, EMI406 to EMI105

Commit message: Update iBOM with exclusions and EMI filters
Parts:
- EMI101, EMI102, EMI103, EMI104, EMI105: value ~ -> 100pF (101)
Changed lines of the file:
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@@
 			)
 		)
-		(property "Value" "~"
+		(property "Value" "100pF (101)"
 			(at 400.05 186.055 0)
 			(effects
@@
 			)
 		)
-		(property "Value" "~"
+		(property "Value" "100pF (101)"
 			(at 381 188.595 0)
 			(effects
@@
 			)
 		)
-		(property "Value" "~"
+		(property "Value" "100pF (101)"
 			(at 332.74 225.425 0)
 			(effects
@@
 			)
 		)
-		(property "Value" "~"
+		(property "Value" "100pF (101)"
 			(at 494.03 191.135 0)
 			(effects
@@
 			)
 		)
-		(property "Value" "~"
+		(property "Value" "100pF (101)"
 			(at 311.15 220.345 0)
 			(effects
