File: 312628-REV-6C/sheets/PRINTER_SERIAL.kicad_sch (KiCad schematic)
At the start: 88 parts, among them CN401 DB25, CN402 DB25, Q401 2N3904, U401 MSM6242B, U402 8250, U403 PPC1, U404 MC1488, U405 MC1489

Commit message: Update Schematics to KiCad V8
Parts:
- renumbered C202 to C401, C202 to C404, C202 to C405, C202 to C406, C202 to C408, C202 to C409, C202 to C410, C202 to C411, C202 to C412, C202 to C413, C202 to C414, C202 to C415, C202 to C416, C202 to C417, C202 to C418, C202 to C419, C202 to C420, C202 to C421, C202 to C422, C202 to C423, C202 to C424, C202 to C757, C202 to C760, C202 to C761, C202 to C762, C202 to C776, CR201 to CR401, CR201 to CR402, CR201 to CR403, CR201 to CR404, CR201 to CR405, R206 to R401, R206 to R402, R206 to R403, R206 to R404, R206 to R405, R206 to R407, R206 to R408, R206 to R409, R206 to R410, R206 to R411, R206 to R412, R206 to R413, R206 to R414, R206 to R421

Commit message: Update iBOM with exclusions and EMI filters
Parts:
- D690, JMP690: now left out of the parts list
- EMI401, EMI402, EMI403, EMI404, EMI405, EMI406, EMI407, EMI408, EMI409, EMI410, EMI411, EMI412, EMI413, EMI414, EMI415, EMI416, EMI417, EMI418, EMI419, EMI420, EMI421, EMI422, EMI423, EMI424, EMI425: value ~ -> 100pF (101)
- XTAL2: value 32.XXKHZ -> 32.768KHZ
Changed lines of the file:
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@@
 			)
 		)
-		(property "Value" "~"
+		(property "Value" "100pF (101)"
 			(at 371.475 90.805 0)
 			(effects
@@
 			)
 		)
-		(property "Value" "~"
+		(property "Value" "100pF (101)"
 			(at 526.415 190.5 0)
 			(effects
@@
 			)
 		)
-		(property "Value" "~"
+		(property "Value" "100pF (101)"
 			(at 470.535 285.75 0)
 			(effects
@@
 			)
 		)
-		(property "Value" "~"
+		(property "Value" "100pF (101)"
 			(at 332.74 66.04 0)
 			(effects
@@
 			)
 		)
-		(property "Value" "~"
+		(property "Value" "100pF (101)"
 			(at 344.805 73.66 0)
 			(effects
@@
 			)
 		)
-		(property "Value" "~"
+		(property "Value" "100pF (101)"
 			(at 387.35 97.79 0)
 			(effects
@@
 			)
 		)
-		(property "Value" "~"
+		(property "Value" "100pF (101)"
 			(at 277.495 30.48 0)
 			(effects
@@
 		(unit 1)
 		(exclude_from_sim no)
-		(in_bom yes)
+		(in_bom no)
 		(on_board yes)
 		(dnp no)
@@
 			)
 		)
-		(property "Value" "~"
+		(property "Value" "100pF (101)"
 			(at 423.545 327.66 0)
 			(effects
@@
 			)
 		)
-		(property "Value" "~"
+		(property "Value" "100pF (101)"
 			(at 316.23 54.61 0)
 			(effects
@@
 		(unit 1)
 		(exclude_from_sim no)
-		(in_bom yes)
+		(in_bom no)
 		(on_board yes)
 		(dnp no)
@@
 			)
 		)
-		(property "Value" "~"
+		(property "Value" "100pF (101)"
 			(at 484.505 166.37 0)
 			(effects
@@
 			)
 		)
-		(property "Value" "~"
+		(property "Value" "100pF (101)"
 			(at 503.555 259.08 0)
 			(effects
@@
 			)
 		)
-		(property "Value" "~"
+		(property "Value" "100pF (101)"
 			(at 290.195 38.1 0)
 			(effects
@@
 			)
 		)
-		(property "Datasheet" " ~"
+		(property "Datasheet" "~"
 			(at 565.785 283.845 0)
 			(effects
@@
 			)
 		)
-		(property "Value" "~"
+		(property "Value" "100pF (101)"
 			(at 455.295 298.45 0)
 			(effects
@@
 			)
 		)
-		(property "Value" "~"
+		(property "Value" "100pF (101)"
 			(at 426.085 122.555 0)
 			(effects
@@
 			)
 		)
-		(property "Value" "~"
+		(property "Value" "100pF (101)"
 			(at 497.205 173.99 0)
 			(effects
@@
 			)
 		)
-		(property "Value" "~"
+		(property "Value" "100pF (101)"
 			(at 405.765 342.9 0)
 			(effects
@@
 			)
 		)
-		(property "Value" "~"
+		(property "Value" "100pF (101)"
 			(at 471.805 158.75 0)
 			(effects
@@
 			)
 		)
-		(property "Value" "~"
+		(property "Value" "100pF (101)"
 			(at 516.255 246.38 0)
 			(effects
@@
 			)
 		)
-		(property "Value" "~"
+		(property "Value" "100pF (101)"
 			(at 441.325 313.69 0)
 			(effects
@@
 			)
 		)
-		(property "Value" "32.XXKHZ"
+		(property "Value" "32.768KHZ"
 			(at 90.805 62.23 0)
 			(effects
@@
 			)
 		)
-		(property "Value" "~"
+		(property "Value" "100pF (101)"
 			(at 412.115 113.665 0)
 			(effects
@@
 			)
 		)
-		(property "Value" "~"
+		(property "Value" "100pF (101)"
 			(at 511.175 182.88 0)
 			(effects
@@
 			)
 		)
-		(property "Value" "~"
+		(property "Value" "100pF (101)"
 			(at 399.415 105.41 0)
 			(effects
@@
 			)
 		)
-		(property "Value" "~"
+		(property "Value" "100pF (101)"
 			(at 302.26 45.72 0)
 			(effects
@@
 			)
 		)
-		(property "Datasheet" " ~"
+		(property "Datasheet" "~"
 			(at 564.515 121.285 0)
 			(effects
@@
 			)
 		)
-		(property "Value" "~"
+		(property "Value" "100pF (101)"
 			(at 357.505 81.915 0)
 			(effects
@@
 			)
 		)
-		(property "Value" "~"
+		(property "Value" "100pF (101)"
 			(at 487.045 271.78 0)
 			(effects
