File: 312628-REV-6C/sheets/VIDEO.kicad_sch (KiCad schematic)
At the start: 89 parts, among them CN203 Jumper_2_Open, CN601 DB 9, CN602 DB 9, CN603 "RCA" Jack, Q601 2N3904, Q602 2N3906, U1 74LS04, U111 74LS125, U601 PVC4, U602 CSG 5720, U603 74LS244, U604 74LS245, U605 4464, U606 4464, U607 CHAR-ROM

Commit message: Update Schematics to KiCad V8
Parts:
- renumbered C202 to C601, C202 to C602, C202 to C603, C202 to C604, C202 to C605, C202 to C606, C202 to C607, C202 to C608, C202 to C609, C202 to C610, C202 to C613, C202 to C766, C202 to C767, C202 to C768, C202 to C769, C202 to C770, C202 to C802, C202 to C803, CR201 to CR601, EMI412 to EMI607, EMI412 to EMI608, EMI412 to EMI609, EMI412 to EMI610, EMI412 to EMI611, EMI412 to EMI612, EMI412 to EMI613, EMI412 to EMI614, FB201 to FB602, FB201 to FB603, FB201 to FB604, FB201 to FB605, FB201 to FB606, FB201 to FB607, FB201 to FB608, FB201 to FB609, FB201 to FB610, FB201 to FB611, CN203 to JMP611, CN203 to JMP612, CN203 to JMP614, R206 to R601, R206 to R602, R206 to R603, R206 to R604, R206 to R605, R206 to R606, R206 to R607, R206 to R608, R206 to R616, R206 to R617, R206 to R618, R206 to R619, R206 to R620, R206 to R622, R206 to R623, R206 to R624, R206 to R625, R206 to R626, R206 to R627, R206 to R628, R206 to R629, R206 to R630, R206 to R639, R206 to R640, R206 to R641, R206 to R642, R206 to R643, R206 to R645, RP402 to RP602
Connections:
- net SW1: now also U1.13; no longer U1.9
- net at U607.23 (A11): now also U1.12; no longer U1.8

Commit message: Update iBOM with exclusions and EMI filters
Parts:
- EMI607, EMI608, EMI609, EMI610, EMI611, EMI612, EMI613, EMI614: value ~ -> 100pF (101)
- OSC602: now left out of the parts list
Changed lines of the file:
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@@
 			)
 		)
-		(property "Value" "~"
+		(property "Value" "100pF (101)"
 			(at 499.11 236.855 0)
 			(effects
@@
 			)
 		)
-		(property "Value" "~"
+		(property "Value" "100pF (101)"
 			(at 486.41 234.315 0)
 			(effects
@@
 			)
 		)
-		(property "Datasheet" " ~"
+		(property "Datasheet" "~"
 			(at 376.555 67.31 0)
 			(effects
@@
 			)
 		)
-		(property "Value" "~"
+		(property "Value" "100pF (101)"
 			(at 431.8 193.675 0)
 			(effects
@@
 			)
 		)
-		(property "Value" "~"
+		(property "Value" "100pF (101)"
 			(at 473.71 231.775 0)
 			(effects
@@
 			)
 		)
-		(property "Value" "~"
+		(property "Value" "100pF (101)"
 			(at 511.81 239.395 0)
 			(effects
@@
 			)
 		)
-		(property "Datasheet" " ~"
+		(property "Datasheet" "~"
 			(at 450.85 195.58 0)
 			(effects
@@
 			)
 		)
-		(property "Value" "~"
+		(property "Value" "100pF (101)"
 			(at 473.71 265.43 0)
 			(effects
@@
 			)
 		)
-		(property "Value" "~"
+		(property "Value" "100pF (101)"
 			(at 486.41 267.97 0)
 			(effects
@@
 			)
 		)
-		(property "Value" "~"
+		(property "Value" "100pF (101)"
 			(at 499.11 270.51 0)
 			(effects
@@
 			)
 		)
-		(property "Datasheet" " ~"
+		(property "Datasheet" "~"
 			(at 546.1 259.08 0)
 			(effects
@@
 		(unit 1)
 		(exclude_from_sim no)
-		(in_bom yes)
+		(in_bom no)
 		(on_board yes)
 		(dnp no)
